Commit message: Cleanup.

File: urdf/materials.xacro (robot description, xacro)
@@ -4,3 +4,12 @@
   <color rgba="0.700 0.700 0.700 1.000"/>
 </material>
+    <material name="blue">
+        <color rgba="0 0 0.8 1"/>
+    </material>
+    <material name="black">
+        <color rgba="0 0 0 1"/>
+    </material>
+    <material name="white">
+        <color rgba="1 1 1 1"/>
+    </material>
 </robot>

File: urdf/robot.xacro.urdf (robot description, URDF)
Before this commit: robot diff_drive, 7 links, 6 joints
Links:
- removed link caster
- removed link chassis_link
- removed link gnss_link
- removed link imu_link
- removed link left_wheel
- removed link right_wheel
- added link front_left, mass 23.230413890431347; collision mesh filename=file://$(find nav2_outdoor_example)/urdf/meshes/wheel_4_1.s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 scale=0.001 0.001 0.001; visual mesh filename=file://$(find nav2_outdoor_example)/urdf/meshes/wheel_4_1.s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 scale=0.001 0.001 0.001
- added link front_right, mass 23.230413890431347; collision mesh filename=file://$(find nav2_outdoor_example)/urdf/meshes/wheel_3_1.s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 scale=0.001 0.001 0.001; visual mesh filename=file://$(find nav2_outdoor_example)/urdf/meshes/wheel_3_1.s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 scale=0.001 0.001 0.001
- added link rear_left, mass 23.230413890431347; collision mesh filename=file://$(find nav2_outdoor_example)/urdf/meshes/wheel_2_1.s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 scale=0.001 0.001 0.001; visual mesh filename=file://$(find nav2_outdoor_example)/urdf/meshes/wheel_2_1.s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 scale=0.001 0.001 0.001
- added link rear_right, mass 23.230413890431347; collision mesh filename=file://$(find nav2_outdoor_example)/urdf/meshes/wheel_1_1.s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 scale=0.001 0.001 0.001; visual mesh filename=file://$(find nav2_outdoor_example)/urdf/meshes/wheel_1_1.s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 scale=0.001 0.001 0.001
- link base_link: mass None -> 97.36517446475621; geometry collision mesh filename=file://$(find nav2_outdoor_example)/urdf/meshes/base_link.s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 scale=0.001 0.001 0.001; visual mesh filename=file://$(find nav2_outdoor_example)/urdf/meshes/base_link.s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 scale=0.001 0.001 0.001
Joints:
- removed joint caster_joint
- removed joint chassis_joint
- removed joint gnss_joint
- removed joint imu_joint
- removed joint left_wheel_joint
- removed joint right_wheel_joint
- added joint front_left_joint: type continuous, parent base_link, child front_left, origin xyz=0.35 0.233285 0.0 rpy=0 0 0, axis 0.5 0.866025 0.0
- added joint front_right_joint: type continuous, parent base_link, child front_right, origin xyz=0.35 -0.233285 0.0 rpy=0 0 0, axis -0.5 0.866025 -0.0
- added joint rear_left_joint: type continuous, parent base_link, child rear_left, origin xyz=-0.35 0.233285 0.0 rpy=0 0 0, axis -0.5 0.866025 0.0
- added joint rear_right_joint: type continuous, parent base_link, child rear_right, origin xyz=-0.35 -0.233285 0.0 rpy=0 0 0, axis 0.5 0.866025 -0.0
