Commit message: Shift IMU.

File: urdf/robot.xacro.urdf (robot description, URDF)
Before this commit: robot diff_drive, 7 links, 6 joints
Joints:
- joint chassis_joint: origin (none) -> xyz=-0.554283 0 0 rpy=0 0 0

Commit message: Rotated IMU.

File: urdf/robot.xacro.urdf (robot description, URDF)
Before this commit: robot diff_drive, 7 links, 6 joints
Joints:
- joint imu_joint: origin xyz=0.554283 0 1.0 rpy=0 0 0 -> xyz=0.554283 0 1.0 rpy=0 0 1.57

Commit message: Arbitrary oriented IMU.

File: urdf/robot.xacro.urdf (robot description, URDF)
Before this commit: robot diff_drive, 7 links, 6 joints
Joints:
- joint imu_joint: origin xyz=0.554283 0 1.0 rpy=0 0 1.57 -> xyz=0.554283 0 1.0 rpy=0.5 1.2 -1.17

Commit message: Add GPS and IMU

File: urdf/robot.xacro.urdf (robot description, URDF)
Before this commit: robot diff_drive, 5 links, 4 joints
Links:
- added link gnss_link, mass 0.005; collision sphere radius=0.05; visual sphere radius=0.05
- added link imu_link, mass 0.005; collision sphere radius=0.05; visual sphere radius=0.05
Joints:
- added joint gnss_joint: type fixed, parent base_link, child gnss_link, origin xyz=0 0 -0.05 rpy=0 0 0
- added joint imu_joint: type fixed, parent base_link, child imu_link, origin xyz=0 0 0.05 rpy=0.5 1.2 -1.17

Commit message: Rotate links of wheels.

File: urdf/robot.xacro.urdf (robot description, URDF)
Before this commit: robot diff_drive, 7 links, 6 joints
Joints:
- joint front_left_joint: origin xyz=0.35 0.233285 0.0 rpy=0 0 0 -> xyz=0.35 0.233285 0.0 rpy=0 0 -2.07079698039
- joint front_right_joint: origin xyz=0.35 -0.233285 0.0 rpy=0 0 0 -> xyz=0.35 -0.233285 0.0 rpy=0 0 2.07079698039
- joint rear_left_joint: origin xyz=-0.35 0.233285 0.0 rpy=0 0 0 -> xyz=-0.35 0.233285 0.0 rpy=0 0 -1.07079566641 
- joint rear_right_joint: origin xyz=-0.35 -0.233285 0.0 rpy=0 0 0 -> xyz=-0.35 -0.233285 0.0 rpy=0 0 1.07079566641

Commit message: Simplify launch.

File: urdf/robot.xacro.urdf (robot description, URDF)
Before this commit: robot diff_drive, 7 links, 6 joints
Links:
- link front_left: geometry collision mesh filename=file://$(find nav2_outdoor_example)/urdf/meshes/wheel.stl scale=0.001 0.001 0.001; visual mesh filename=file://$(find nav2_outdoor_example)/urdf/meshes/wheel.stl scale=0.001 0.001 0.001
- link front_right: geometry collision mesh filename=file://$(find nav2_outdoor_example)/urdf/meshes/wheel.stl scale=0.001 0.001 0.001; visual mesh filename=file://$(find nav2_outdoor_example)/urdf/meshes/wheel.stl scale=0.001 0.001 0.001
- link rear_left: geometry collision mesh filename=file://$(find nav2_outdoor_example)/urdf/meshes/wheel.stl scale=0.001 0.001 0.001; visual mesh filename=file://$(find nav2_outdoor_example)/urdf/meshes/wheel.stl scale=0.001 0.001 0.001
- link rear_right: geometry collision mesh filename=file://$(find nav2_outdoor_example)/urdf/meshes/wheel.stl scale=0.001 0.001 0.001; visual mesh filename=file://$(find nav2_outdoor_example)/urdf/meshes/wheel.stl scale=0.001 0.001 0.001
Joints:
- joint front_left_joint: axis 0.5 0.866025 0.0 -> -1 0 0
- joint front_right_joint: axis -0.5 0.866025 -0.0 -> 1 0 0
- joint rear_left_joint: axis -0.5 0.866025 0.0 -> -1 0 0
- joint rear_right_joint: axis 0.5 0.866025 -0.0 -> 1 0 0

Commit message: Use xacro to create wheels.

File: urdf/robot.xacro.urdf (robot description, URDF)
Before this commit: robot diff_drive, 7 links, 6 joints
Links:
- removed link front_left
- removed link front_right
- removed link rear_left
- removed link rear_right
Joints:
- removed joint front_left_joint
- removed joint front_right_joint
- removed joint rear_left_joint
- removed joint rear_right_joint
